Commit message: 留存

File: .localization_fix_backups/20260817_142102/src/unitree_guide/unitree_ros/robots/a1_description/xacro/gazebo.xacro (robot description, xacro)
@@ -341,13 +341,7 @@
                     </ray>
                     <visualize>false</visualize>
-                    <!-- Trace 1200 deterministic full-FOV rays per update.
-                         Denser snapshots over-correlate planar constraints
-                         and destabilize FAST-LIO in corridors. -->
+                    <!-- Keep the original 24 ms Livox scan phase while tracing 1200 rays. -->
                     <samples>2400</samples>
                     <downsample>2</downsample>
-                    <!-- Use a deterministic full-FOV ray subset at 10 Hz.
-                         FAST-LIO otherwise receives nearly disjoint sparse
-                         pattern fragments and its first scan match diverges. -->
-                    <stable_full_scan>true</stable_full_scan>
                     <csv_file_name>package://a1_description/scan_mode/mid360.csv</csv_file_name>
                     <ros_topic>/scan</ros_topic>

File: .localization_fix_backups/20260817_142102/src/unitree_guide/unitree_ros/robots/a1_description/xacro/robot.xacro (robot description, xacro)
@@ -118,9 +118,6 @@
         </collision>
     </link>
-    <!-- Keep the physical Mid-360 body at the repository's original pose.
-         Its collision mesh must not be rotated as a side effect of changing
-         the localization scan extrinsics, otherwise Gazebo contact dynamics
-         (and therefore the stand-up motion) can change. -->
-    <link name="laser_livox_body">
+    <!-- livox mid360 -->
+    <link name="laser_livox">
             <collision>
                 <origin xyz="0 0 0" rpy="0 0 0"/>
@@ -136,16 +133,7 @@
             </visual>
     </link>
-    <joint name="laser_livox_body_joint" type="fixed">
+    <joint name="laser_livox_joint" type="fixed">
             <origin xyz="0.2 0 0.08" rpy="0 0.785 0"/>
             <parent link="base"/>
-            <child link="laser_livox_body"/>
-    </joint>
-    <!-- Collision-free scan frame.  The ray sensor is mounted here so the
-         localization point cloud stays level without modifying the physical
-         lidar body or the robot's collision geometry. -->
-    <link name="laser_livox"/>
-    <joint name="laser_livox_joint" type="fixed">
-            <origin xyz="0.2 0 0.08" rpy="0 0 0"/>
-            <parent link="base"/>
             <child link="laser_livox"/>
     </joint>
@@ -171,6 +159,5 @@
     </link>
     <joint name="livox_imu_joint" type="fixed">
-            <!-- Preserve the original physical IMU mounting orientation. -->
-            <parent link="laser_livox_body"/>
+            <parent link="laser_livox"/>
             <child link="livox_imu_link"/>
             <origin rpy="0 0 0" xyz="-0.011 -0.02329 0.04412"/>
